File: hardware/AudioAmpV1.kicad_pcb (KiCad board)
At the start: 4 copper layers, 52.1 x 75.1 mm, 45 parts, among them J1 3,5mm Jack, J2 Barrel_Jack_Switch, J3 Speaker_R, J4 Speaker_L, U1 PAM8610

Commit message: Add files via upload
Parts:
- moved G*** 0.63 mm to (152.8, 114.5)
